File: BQ76952_uPi_Hat.kicad_sch (KiCad schematic)
At the start: 90 parts, among them J1 GPIO, J2 61202021621, P1 61302421121, P2 61300821121, P3 61300421121, Q1 FCX495TA, Q2 2N7002, SW1 416131160801, U1 PBQ76952PFBT, U2 LM317DCY, U3 STM1061N38WX6F

Commit message: updating outdating files
Parts:
- C1, C10, C11, C12, C13, C14, C15, C16, C18, C19, C2, C20, C21, C22, C23, C24, C25, C26, C27, C28, C29, C3, C4, C6, C7, C8, C9: symbol Device:C_Small -> Symbol Library:C_Small
- C17, C5: symbol Device:C_Polarized -> Symbol Library:C_Polarized
- D1, D3: symbol Diode:1N4002 -> Symbol Library:1N4002
- D10, D4, D5, D6, D7, D8: symbol Device:LED -> Symbol Library:LED
- D2, D9: symbol Device:D_Schottky -> Symbol Library:D_Schottky
- H1, H2, H3, H4: symbol Mechanical:MountingHole -> Symbol Library:MountingHole
- J1: symbol Connector_Generic:Conn_02x20_Odd_Even -> Symbol Library:Conn_02x20_Odd_Even
- J2: symbol WR-BHD 1.27 mm Male:62702021721 -> Symbol Library:62702021721
- P1: symbol WR_PHD 2.54 Dual Male:61302421121 -> Symbol Library:61302421121
- P2: symbol WR_PHD 2.54 Dual Male:61300821121 -> Symbol Library:61300821121
- P3: symbol WR_PHD 2.54 Dual Male:61300421121 -> Symbol Library:61300421121
- Q1: symbol FCX495TA:FCX495TA -> Symbol Library:FCX495TA
- Q2: symbol Transistor_FET:2N7002 -> Symbol Library:2N7002
- R1, R10, R11, R12, R13, R14, R15, R16, R17, R18, R19, R2, R20, R21, R22, R23, R24, R25, R26, R27, R28, R29, R3, R30, R31, R32, R33, R34, R35, R36, R4, R5, R6, R7, R8, R9: symbol Device:R -> Symbol Library:R
- SW1: symbol Switch:SW_DIP_x01 -> Symbol Library:SW_DIP_x01
- U1: symbol BQ76952:PBQ76952PFBT -> Symbol Library:PBQ76952PFBT
- U2: symbol LM317DCY:LM317DCY -> Symbol Library:LM317DCY
- U3: symbol STM1061N38WX6F:STM1061N38WX6F -> Symbol Library:STM1061N38WX6F
